Commit message: Adjusted robot dimensions

File: meteron_mocup/mocup_description/urdf/mocup_parameters.urdf.xacro (robot description, xacro)
@@ -6,6 +6,6 @@
   <xacro:property name="wheel_suspension_offset_y" value="0.1435" />
   <xacro:property name="wheel_suspension_offset_z" value="0" />
-  <xacro:property name="wheel_radius" value="0.03" />
-  <xacro:property name="wheel_size_y" value="0.04" />
+  <xacro:property name="wheel_radius" value="0.035" />
+  <xacro:property name="wheel_size_y" value="0.035" />
   <xacro:property name="wheel_offset_x" value="0" />
   <xacro:property name="wheel_offset_y" value="-0.0055" />

File: meteron_mocup/mocup_gazebo/urdf/mocup_base_controllers.urdf.xacro (robot description, xacro)
@@ -6,5 +6,5 @@
     <plugin name="all_wheel_steering_controller" filename="liball_wheel_steering_plugin.so">
       <alwaysOn>true</alwaysOn>
-      <controlRate>1000.0</controlRate>
+      <controlRate>50.0</controlRate>
       <updateRate>0.0</updateRate>
       <frontLeftAxle>front_left_wheel_joint</frontLeftAxle>
@@ -20,11 +20,10 @@
       <rearLeftJoint>rear_left_wheel_suspension_joint</rearLeftJoint>
       <rearRightJoint>rear_right_wheel_suspension_joint</rearRightJoint>
-      <wheelTrack>0.287</wheelTrack>
-      <wheelBase>0.3</wheelBase>
-      <wheelRadius>0.03</wheelRadius>
+      <wheelBase>0.30</wheelBase>
+      <wheelTrack>0.305</wheelTrack>
+      <wheelRadius>0.035</wheelRadius>
       <jointMaxTorque>10</jointMaxTorque>
-      <wheelMaxTorque>1</wheelMaxTorque>
-      <minRadius>0.4</minRadius>
-      <maxVelX>1.0</maxVelX>
+      <wheelMaxTorque>10</wheelMaxTorque>
+      <maxVelX>0.1</maxVelX>
       <robotNamespace>/</robotNamespace>
       <topicName>drive</topicName>
@@ -33,7 +32,7 @@
     <plugin name="p3d_base_controller" filename="libgazebo_ros_p3d.so">
       <alwaysOn>true</alwaysOn>
-      <updateRate>1000.0</updateRate>
+      <updateRate>50.0</updateRate>
       <bodyName>base_link</bodyName>
-      <topicName>state</topicName>
+      <topicName>/ground_truth/state</topicName>
       <gaussianNoise>0.01</gaussianNoise>
       <xyzOffsets>0 0 0</xyzOffsets>
@@ -43,5 +42,5 @@
       <plugin name="camera_servo_controller" filename="libhector_servo_plugin.so">
         <alwaysOn>true</alwaysOn>
-        <controlRate>1000.0</controlRate>
+        <controlRate>50.0</controlRate>
         <updateRate>0.0</updateRate>
         <firstServoName>camera/z</firstServoName>
