Commit message: Cleaned code

File: meteron_mocup/mocup_description/urdf/mocup_camera_mast.urdf.xacro (robot description, xacro)
@@ -8,5 +8,5 @@
       <child link="camera_mast_link" />
       <axis xyz="0 0 1" />
-      <limit lower="${-M_PI}" upper="${M_PI}" effort="100" velocity="100" />
+      <limit lower="${-2*M_PI}" upper="${2*M_PI}" effort="100" velocity="100" />
     </joint>
     <link name="camera_mast_link">

File: meteron_mocup/mocup_gazebo/urdf/mocup_base_controllers.urdf.xacro (robot description, xacro)
@@ -34,5 +34,5 @@
       <updateRate>50.0</updateRate>
       <bodyName>base_link</bodyName>
-      <topicName>/ground_truth/state</topicName>
+      <topicName>state</topicName>
       <gaussianNoise>0.01</gaussianNoise>
       <xyzOffsets>0 0 0</xyzOffsets>
