Commit message: improvements and bugfixes

File: meteron_mocup/mocup_gazebo/urdf/mocup_base_controllers.urdf.xacro (robot description, xacro)
@@ -25,5 +25,5 @@
       <jointMaxTorque>10</jointMaxTorque>
       <wheelMaxTorque>10</wheelMaxTorque>
-      <jointMaxVelocity>0.0</jointMaxVelocity>
+      <jointMaxVelocity>0.33</jointMaxVelocity>
       <maxVelX>0.1</maxVelX>
       <robotNamespace>/</robotNamespace>

File: meteron_mocup/mocup_gazebo/urdf/mocup_gazebo.urdf.xacro (robot description, xacro)
@@ -2,12 +2,5 @@
 <robot xmlns:xacro="http://ros.org/wiki/xacro"
        name="mocup">
-  <xacro:include filename="$(find mocup_description)/urdf/mocup_parameters.urdf.xacro" />
-  <xacro:include filename="$(find mocup_description)/urdf/materials.urdf.xacro" />
-  <xacro:include filename="$(find mocup_description)/urdf/mocup_base.urdf.xacro" />
-  <xacro:mocup_base wheel_joint_type="continuous" />
-  <xacro:include filename="$(find hector_sensors_description)/urdf/asus_camera.urdf.xacro" />
-    <xacro:asus_camera name="camera" parent="camera_base_link">
-      <origin xyz="0.0 0.0 0.0" rpy="0 0 0"/>
-    </xacro:asus_camera>
+  <xacro:include filename="$(find mocup_description)/urdf/mocup.urdf.xacro" />
   <xacro:include filename="$(find mocup_gazebo)/urdf/mocup_base_controllers.urdf.xacro" />
   <xacro:mocup_base_controllers/>
